Commit message: rviz and launch donezo

File: qube_description/urdf/qube.urdf.xacro (robot description, xacro)
@@ -1,10 +1,10 @@
 <?xml version="1.0"?>
-<robot xmlns:xacro="http://www.ros.org/wiki/xacro" >
+<robot name="qube" xmlns:xacro="http://www.ros.org/wiki/xacro" >
 	<xacro:include filename="$(find qube_description)/urdf/qube.macro.xacro" />
     <link name="world"/>
-    <xacro:joint_model prefix="qube" />
-	<joint name="${prefix}base_joint" type="fixed">
+    <xacro:joint_model prefix="" />
+	<joint name="base_joint" type="fixed">
         <parent link="world"/>
-        <child link="qubebase_link"/>
+        <child link="base_link"/>
     </joint>
 </robot>
