Commit message: dokumenterte, ryddet, og la til en selvevaluering

File: install/qube_bringup/share/qube_bringup/urdf/controlled_qube.urdf.xacro (robot description, xacro)
@@ -1,18 +1,19 @@
 <?xml version="1.0"?>
 <robot name="qube" xmlns:xacro="http://www.ros.org/wiki/xacro">
+    <!-- Definere argumenter for hardware parameter -->
     <xacro:arg name="baud_rate" default="115200"/>
     <xacro:arg name="device" default="/dev/ttyACM0"/>
     <xacro:arg name="simulation" default="true"/>
-    <!-- Include existing Qube components -->
+    <!-- Inkludere qube komponenter (xacro maxroen fra qube_description), og driver fra Lars Ivar sitt bibliotek -->
     <xacro:include filename="$(find qube_description)/urdf/qube.macro.xacro" />
     <xacro:include filename="$(find qube_driver)/ros2_control/qube_driver.ros2_control.xacro" />
-    <!-- Base link and world connection -->
+    <!-- Sette opp verden og legge in en qube fra makroen -->
     <link name="world"/>
-    <xacro:joint_model prefix="" />
+    <xacro:qube_model prefix="" />
     <joint name="base_joint" type="fixed">
         <parent link="world"/>
         <child link="base_link"/>
     </joint>
-    <!-- ROS2 Control integration -->
+    <!-- Sette opp Lars Ivar sin driver og sende argumenter -->
     <xacro:qube_driver_ros2_control
         name="qube_driver"

File: install/qube_description/share/qube_description/urdf/qube.macro.xacro (robot description, xacro)
@@ -5,5 +5,6 @@
   <xacro:property name="disk_thickness" value="0.01" />
   <xacro:property name="dial_thickness" value="0.002" />
-  <xacro:macro name="joint_model" params="prefix">
+  <!-- Macro for hele quben -->
+  <xacro:macro name="qube_model" params="prefix">
     <!-- Materials -->
     <material name="${prefix}black">
@@ -16,4 +17,5 @@
       <color rgba="1 0 0 1"/>
     </material>
+    <!-- Links og joints for hele basen -->
     <link name="${prefix}base_link"/>
     <joint name="${prefix}stator_joint" type="fixed">
@@ -30,4 +32,5 @@
       </visual>
     </link>
+    <!-- joint for å koble rorten til basen -->
     <joint name="${prefix}motor_joint" type="revolute">
       <parent link="${prefix}stator_link"/>
@@ -37,4 +40,5 @@
       <axis xyz="0 0 1"/>
     </joint>
+    <!-- Links og joints for å lage rotoren -->
     <link name="${prefix}rotor_link">
       <visual>

File: install/qube_description/share/qube_description/urdf/qube.urdf.xacro (robot description, xacro)
@@ -2,6 +2,9 @@
 <robot name="qube" xmlns:xacro="http://www.ros.org/wiki/xacro" >
 	<xacro:include filename="$(find qube_description)/urdf/qube.macro.xacro" />
+    <!-- Lage en world link -->
     <link name="world"/>
-    <xacro:joint_model prefix="" />
+    <!-- Bruke macroen for å lage en qube -->
+    <xacro:qube_model prefix="" />
+    <!-- Koble quben til verden -->
 	<joint name="base_joint" type="fixed">
         <parent link="world"/>
