Commit message: bringup og driver e joever

File: install/qube_description/share/qube_description/urdf/qube.macro.xacro (robot description, xacro)
@@ -30,5 +30,5 @@
       </visual>
     </link>
-    <joint name="${prefix}angle" type="revolute">
+    <joint name="${prefix}motor_joint" type="revolute">
       <parent link="${prefix}stator_link"/>
       <child link="${prefix}rotor_link"/>

Commit message: endre nokke (kanskje)

File: install/qube_description/share/qube_description/urdf/qube.macro.xacro (robot description, xacro)
@@ -35,5 +35,4 @@
       <origin xyz="0 0 ${box_width/2}"/>
       <axis xyz="0 0 1"/>
-      <limit lower="-3.1416" upper="3.1416" effort="10" velocity="10"/>
     </joint>
     <link name="${prefix}rotor_link">

Commit message: funka fjell, men kan gjerne vaskes opp litt (for eksempel å sikre at alle parameter e lett å endre på endten i launchen eller mens den kjøre)

File: install/qube_description/share/qube_description/urdf/qube.macro.xacro (robot description, xacro)
@@ -34,4 +34,5 @@
       <child link="${prefix}rotor_link"/>
       <origin xyz="0 0 ${box_width/2}"/>
+      <limit lower="-3.14" upper="3.14" effort="10" velocity="10"/>
       <axis xyz="0 0 1"/>
     </joint>

Commit message: hvorfor gitignore ikke funka?

File: install/qube_description/share/qube_description/urdf/qube.macro.xacro (robot description, xacro)
@@ -38,5 +38,5 @@
       <origin xyz="0 0 ${box_width/2}"/>
       <limit lower="-3.14" upper="3.14" effort="10" velocity="10"/>
-      <axis xyz="0 0 1"/>
+      <axis xyz="0 0 -1"/>
     </joint>
     <!-- Links og joints for å lage rotoren -->
